File: fpga.kicad_sch (KiCad schematic)
At the start: 6 parts, among them IC1 RP2040_breakout, J6 Micro_SD_Card, U3 CYC1000

Commit message: Version 0.2
Parts:
- IC1: footprint rp2040:RP2040-Breakout -> rp2040:RP2040-Breakout_swd; symbol rp2040-breakout:RP2040_breakout -> rp2040:RP2040_breakout_swd
Connections:
- net GND: now also IC1.44 (GND)
- net RP_RESET: now reaches IC1.30 (RUN)
- net C10_M16 renamed C10_N16
- new net RP_SWDCLK: IC1.43 (SWDCLK)
- new net RP_SWDIO: IC1.42 (SWDIO)
Other:
- title: Calypso - was Atlas -> Calypso
Changed lines of the file:
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@@
   (paper "A4")
   (title_block
-    (title "Calypso - was Atlas")
-    (date "2021-04-17")
-    (rev "1")
+    (title "Calypso")
+    (date "2024-08-10")
+    (rev "0.2")
   )
   (junction (at 231.394 92.202) (diameter 0) (color 0 0 0 0)
@@
   (junction (at 139.446 90.932) (diameter 0) (color 0 0 0 0)
   )
-  (no_connect (at 239.014 33.782))
+  (no_connect (at 230.124 33.782))
   (no_connect (at 129.54 46.228))
-  (no_connect (at 233.934 33.782))
-  (no_connect (at 250.444 56.642))
+  (no_connect (at 232.664 33.782))
+  (no_connect (at 227.584 33.782))
   (no_connect (at 129.54 64.008))
   (no_connect (at 61.976 98.044))
@@
     )
   )
+  (global_label "RP_RESET" (shape input) (at 250.444 56.642 0) (fields_autoplaced)
+    (effects (font (size 1.27 1.27)) (justify left))
+    (property "Intersheet References" "${INTERSHEET_REFS}" (id 0) (at 262.0211 56.5626 0)
+      (effects (font (size 1.27 1.27)) (justify left) hide)
+    )
+  )
   (global_label "C10_C15" (shape input) (at 51.816 98.044 270) (fields_autoplaced)
     (effects (font (size 1.27 1.27)) (justify right))
@@
     )
   )
+  (global_label "RP_SWDIO" (shape input) (at 235.204 33.782 90) (fields_autoplaced)
+    (effects (font (size 1.27 1.27)) (justify left))
+    (property "Intersheet References" "${INTERSHEET_REFS}" (id 0) (at 235.1246 22.084 90)
+      (effects (font (size 1.27 1.27)) (justify left) hide)
+    )
+  )
   (global_label "TDO" (shape input) (at 72.136 78.994 0) (fields_autoplaced)
     (effects (font (size 1.27 1.27)) (justify left))
@@
     )
   )
+  (global_label "RP_SWDCLK" (shape input) (at 237.744 33.782 90) (fields_autoplaced)
+    (effects (font (size 1.27 1.27)) (justify left))
+    (property "Intersheet References" "${INTERSHEET_REFS}" (id 0) (at 237.6646 20.4511 90)
+      (effects (font (size 1.27 1.27)) (justify left) hide)
+    )
+  )
   (global_label "C10_N2" (shape input) (at 72.136 67.564 0) (fields_autoplaced)
     (effects (font (size 1.27 1.27)) (justify left))
@@
     )
   )
-  (global_label "C10_M16" (shape input) (at 31.496 54.864 180) (fields_autoplaced)
-    (effects (font (size 1.27 1.27)) (justify right))
-    (property "Intersheet References" "${INTERSHEET_REFS}" (id 0) (at 20.6447 54.7846 0)
+  (global_label "C10_N16" (shape input) (at 31.496 54.864 180) (fields_autoplaced)
+    (effects (font (size 1.27 1.27)) (justify right))
+    (property "Intersheet References" "${INTERSHEET_REFS}" (id 0) (at 20.7656 54.7846 0)
       (effects (font (size 1.27 1.27)) (justify right) hide)
     )
@@
     )
   )
-  (symbol (lib_id "power:+5V") (at 228.854 33.782 0) (unit 1)
+  (symbol (lib_id "power:+5V") (at 225.044 33.782 0) (unit 1)
     (in_bom yes) (on_board yes)
-    (property "Reference" "#PWR011" (id 0) (at 228.854 37.592 0)
-      (effects (font (size 1.27 1.27)) hide)
-    )
-    (property "Value" "+5V" (id 1) (at 229.235 29.3878 0))
-    (property "Footprint" "" (id 2) (at 228.854 33.782 0)
-      (effects (font (size 1.27 1.27)) hide)
-    )
-    (property "Datasheet" "" (id 3) (at 228.854 33.782 0)
+    (property "Reference" "#PWR011" (id 0) (at 225.044 37.592 0)
+      (effects (font (size 1.27 1.27)) hide)
+    )
+    (property "Value" "+5V" (id 1) (at 225.425 29.3878 0))
+    (property "Footprint" "" (id 2) (at 225.044 33.782 0)
+      (effects (font (size 1.27 1.27)) hide)
+    )
+    (property "Datasheet" "" (id 3) (at 225.044 33.782 0)
       (effects (font (size 1.27 1.27)) hide)
     )
@@
     (pin "2")
   )
-  (symbol (lib_id "rp2040-breakout:RP2040_breakout") (at 233.934 54.102 0) (unit 1)
-    (in_bom yes) (on_board yes) (fields_autoplaced)
-    (property "Reference" "IC1" (id 0) (at 241.0334 32.512 0)
+  (symbol (lib_id "rp2040:RP2040_breakout_swd") (at 233.934 54.102 0) (unit 1)
+    (in_bom yes) (on_board yes)
+    (property "Reference" "IC1" (id 0) (at 248.158 32.766 0)
       (effects (font (size 1.27 1.27)) (justify left))
     )
-    (property "Value" "RP2040_breakout" (id 1) (at 241.0334 35.052 0)
+    (property "Value" "RP2040_breakout" (id 1) (at 247.904 35.56 0)
       (effects (font (size 1.27 1.27)) (justify left))
     )
-    (property "Footprint" "rp2040:RP2040-Breakout" (id 2) (at 239.014 38.862 0)
+    (property "Footprint" "rp2040:RP2040-Breakout_swd" (id 2) (at 239.014 38.862 0)
       (effects (font (size 1.27 1.27)) hide)
     )
@@
     (pin "4")
     (pin "40")
+    (pin "41")
+    (pin "42")
+    (pin "43")
+    (pin "44")
     (pin "5")
     (pin "6")
@@
     (pin "2")
   )
+  (symbol (lib_id "power:GND") (at 240.284 33.782 180) (unit 1)
+    (in_bom yes) (on_board yes)
+    (property "Reference" "#PWR0102" (id 0) (at 240.284 27.432 0)
+      (effects (font (size 1.27 1.27)) hide)
+    )
+    (property "Value" "GND" (id 1) (at 240.157 29.3878 0))
+    (property "Footprint" "" (id 2) (at 240.284 33.782 0)
+      (effects (font (size 1.27 1.27)) hide)
+    )
+    (property "Datasheet" "" (id 3) (at 240.284 33.782 0)
+      (effects (font (size 1.27 1.27)) hide)
+    )
+    (pin "1")
+  )
   (symbol (lib_id "power:GND") (at 172.72 69.088 90) (unit 1)
