File: power.kicad_sch (KiCad schematic)
At the start: 8 parts, among them J7 USB_B_Mini, SW1 SWDPDTBLUE, U1 AMS1117-3.3

Commit message: Version 0.2
Parts:
- added SW2: SW_Push, Button_Switch_THT:SW_PUSH_6mm_H4.3mm, symbol Switch:SW_Push
- R45: value R -> 1K
Connections:
- net GND: now also SW2.2
- net IN_5V: now also SW1.6 (C_2); no longer SW1.4 (NC_2)
- new net RP_RESET: SW2.1
Other:
- title: Calypso - was Atlas -> Calypso
Changed lines of the file:
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@@
   (paper "A4")
   (title_block
-    (title "Calypso - was Atlas")
-    (date "2021-04-17")
-    (rev "1")
+    (title "Calypso")
+    (date "2024-08-10")
+    (rev "0.2")
   )
   (junction (at 116.205 31.75) (diameter 0) (color 0 0 0 0)
@@
   (no_connect (at 52.07 34.29))
   (no_connect (at 52.07 36.83))
-  (no_connect (at 213.36 34.29))
+  (no_connect (at 213.36 39.37))
   (no_connect (at 175.26 34.29))
   (no_connect (at 52.07 31.75))
@@
     )
   )
-  (global_label "IN_5V" (shape input) (at 213.36 39.37 0) (fields_autoplaced)
+  (global_label "RP_RESET" (shape input) (at 189.738 61.976 180) (fields_autoplaced)
+    (effects (font (size 1.27 1.27)) (justify right))
+    (property "Intersheet References" "${INTERSHEET_REFS}" (id 0) (at 178.1609 61.8966 0)
+      (effects (font (size 1.27 1.27)) (justify right) hide)
+    )
+  )
+  (global_label "IN_5V" (shape input) (at 213.36 34.29 0) (fields_autoplaced)
     (effects (font (size 1.27 1.27)) (justify left))
-    (property "Intersheet References" "${INTERSHEET_REFS}" (id 0) (at 220.8852 39.2906 0)
+    (property "Intersheet References" "${INTERSHEET_REFS}" (id 0) (at 220.8852 34.2106 0)
       (effects (font (size 1.27 1.27)) (justify left) hide)
     )
@@
     (pin "1")
   )
+  (symbol (lib_id "power:GND") (at 199.898 61.976 90) (unit 1)
+    (in_bom yes) (on_board yes)
+    (property "Reference" "#PWR013" (id 0) (at 206.248 61.976 0)
+      (effects (font (size 1.27 1.27)) hide)
+    )
+    (property "Value" "GND" (id 1) (at 204.2922 61.849 0))
+    (property "Footprint" "" (id 2) (at 199.898 61.976 0)
+      (effects (font (size 1.27 1.27)) hide)
+    )
+    (property "Datasheet" "" (id 3) (at 199.898 61.976 0)
+      (effects (font (size 1.27 1.27)) hide)
+    )
+    (pin "1")
+  )
   (symbol (lib_id "power:PWR_FLAG") (at 121.92 26.035 0) (unit 1)
     (in_bom yes) (on_board yes)
@@
   )
   (symbol (lib_id "Device:R_Small") (at 217.17 36.83 90) (unit 1)
+    (in_bom yes) (on_board yes)
+    (property "Reference" "R45" (id 0) (at 220.98 38.354 90))
+    (property "Value" "1K" (id 1) (at 217.424 39.116 90))
+    (property "Footprint" "Resistor_SMD:R_1206_3216Metric_Pad1.30x1.75mm_HandSolder" (id 2) (at 217.17 36.83 0)
+      (effects (font (size 1.27 1.27)) hide)
+    )
+    (property "Datasheet" "~" (id 3) (at 217.17 36.83 0)
+      (effects (font (size 1.27 1.27)) hide)
+    )
+    (pin "1")
+    (pin "2")
+  )
+  (symbol (lib_id "Switch:SW_Push") (at 194.818 61.976 0) (unit 1)
     (in_bom yes) (on_board yes) (fields_autoplaced)
-    (property "Reference" "R45" (id 0) (at 217.17 30.48 90))
-    (property "Value" "R" (id 1) (at 217.17 33.02 90))
-    (property "Footprint" "Resistor_SMD:R_1206_3216Metric_Pad1.30x1.75mm_HandSolder" (id 2) (at 217.17 36.83 0)
-      (effects (font (size 1.27 1.27)) hide)
-    )
-    (property "Datasheet" "~" (id 3) (at 217.17 36.83 0)
-      (effects (font (size 1.27 1.27)) hide)
-    )
+    (property "Reference" "SW2" (id 0) (at 194.818 53.848 0))
+    (property "Value" "SW_Push" (id 1) (at 194.818 56.388 0))
+    (property "Footprint" "Button_Switch_THT:SW_PUSH_6mm_H4.3mm" (id 2) (at 194.818 56.896 0)
+      (effects (font (size 1.27 1.27)) hide)
+    )
+    (property "Datasheet" "~" (id 3) (at 194.818 56.896 0)
+      (effects (font (size 1.27 1.27)) hide)
+    )
